File: Keyboard Designs/Schematics/75TH/75TH/untitled.kicad_sch (KiCad schematic)
At the start: 158 parts, among them SW1 Switch, SW10 Switch, SW2 Switch, SW3 Switch, SW4 Switch, SW5 Switch, SW6 Switch, SW7 Switch, SW8 Switch, SW9 Switch

Commit message: Started pcb layout
Parts:
- SW+1, SW-1, SW1, SW10, SW2, SW3, SW4, SW5, SW6, SW7, SW8, SW9, SWDel1, SWDown1, SWEsc1, SWF1, SWF10, SWF11, SWF12, SWF2, SWF3, SWF4, SWF5, SWF6, SWF7, SWF8, SWF9, SWLeft1, SWRight1, SWUp1, SW_'1, SW_,1, SW_.1, SW_/1, SW_;1, SW_A1, SW_B1, SW_C1, SW_D1, SW_E1, SW_F1, SW_G1, SW_H1, SW_I1, SW_J1, SW_K1, SW_L1, SW_M1, SW_N1, SW_O1, SW_P1, SW_Q1, SW_R1, SW_S1, SW_T1, SW_U1, SW_V1, SW_W1, SW_X1, SW_Y1, SW_Z1, SW_[1, SW_]1, SW`1: footprint Button_Switch_Keyboard:SW_Cherry_MX_1.00u_PCB -> marbastlib-mx:SW_MX_1u
- SWBckspc2u1: footprint Button_Switch_Keyboard:SW_Cherry_MX_2.00u_PCB -> marbastlib-mx:SW_MX_1u
- SWCaplck1.75u1: footprint Button_Switch_Keyboard:SW_Cherry_MX_1.75u_PCB -> marbastlib-mx:SW_MX_1.75u
- SWEnter2.25u1, SWLshift2.25u1, SWRshift2.25u1, SWSpc2.25u1: footprint Button_Switch_Keyboard:SW_Cherry_MX_2.25u_PCB -> marbastlib-mx:SW_MX_1u
- SWLCtrl1.25u1, SWLalt1.25u1, SWLwin1.25u1, SWRalt1.25u1, SWRwin1.25u1: footprint Button_Switch_Keyboard:SW_Cherry_MX_1.25u_PCB -> marbastlib-mx:SW_MX_1.25u
- SWSpc1.25u1: renamed from SWSpc1u1; footprint Button_Switch_Keyboard:SW_Cherry_MX_1.00u_PCB -> marbastlib-mx:SW_MX_1.25u
- SWSpc2.75u1: footprint Button_Switch_Keyboard:SW_Cherry_MX_2.75u_PCB -> marbastlib-mx:SW_MX_1u
- SWTab1.5u1, SW_\1.5u1: footprint Button_Switch_Keyboard:SW_Cherry_MX_1.50u_PCB -> marbastlib-mx:SW_MX_1.5u
Connections:
- net Column 0 renamed Col 0
- net Column 1 renamed Col 1
- net Column 10 renamed Col 10
- net Column 11 renamed Col 11
- net Column 12 renamed Col 12
- net Column 13 renamed Col 13
- net Column 14 renamed Col 14
- net Col 14: no longer SWDown1.1, SWRight1.1, SWUp1.1
- net Column 2 renamed Col 2
- net Column 3 renamed Col 3
- net Column 4 renamed Col 4
- net Column 5 renamed Col 5
- net Column 6 renamed Col 6
- net Column 7 renamed Col 7
- net Column 8 renamed Col 8
- net Column 9 renamed Col 9
- new net Col 15: SWDown1.1, SWUp1.1
- new net Col 16: SWRight1.1

Commit message: wired usbc and partial MCU
Parts:
- renumbered D67 to D10, D73 to D11, D79 to D12, D85 to D13, D5 to D14, D6 to D15, D7 to D16, D8 to D17, D26 to D18, D32 to D19, D3 to D2, D38 to D20, D44 to D21, D50 to D22, D56 to D23, D62 to D24, D68 to D25, D74 to D26, D86 to D27, D9 to D28, D11 to D29, D4 to D3, D12 to D30, D27 to D31, D33 to D32, D39 to D33, D45 to D34, D51 to D35, D57 to D36, D63 to D37, D69 to D38, D75 to D39, D25 to D4, D81 to D40, D87 to D41, D13 to D42, D19 to D43, D22 to D44, D28 to D45, D34 to D46, D40 to D47, D46 to D48, D52 to D49, D31 to D5, D58 to D50, D64 to D51, D70 to D52, D76 to D53, D82 to D54, D17 to D55, D20 to D56, D23 to D57, D29 to D58, D35 to D59, D43 to D6, D41 to D60, D47 to D61, D53 to D62, D59 to D63, D65 to D64, D71 to D65, D83 to D66, D95 to D67, D15 to D68, D18 to D69, D49 to D7, D24 to D70, D30 to D71, D42 to D72, D54 to D73, D66 to D74, D72 to D75, D84 to D76, D90 to D77, D96 to D78, D2 to D79, D55 to D8, D61 to D9, SW9 to SW10, SW10 to SW11, SW1 to SW2, SW2 to SW3, SW3 to SW4, SW4 to SW5, SW5 to SW6, SW6 to SW7, SW7 to SW8, SW8 to SW9
