File: Keyboard Designs/Schematics/75TH/75TH/75TH.kicad_pcb (KiCad board)
At the start: 2 copper layers, 184 parts, among them J1 OLED_128x64, J2 USB_C_Receptacle_USB2.0_14P, SW1 Switch, SW10 Switch, SW11 RotaryEncoder_Switch_EC11E092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, SW2 Switch, SW3 Switch, SW4 Switch, SW5 Switch, SW6 Switch, SW7 Switch, SW8 Switch, SW9 Switch, U2 STM32F072CBTx

Commit message: wired usbc and partial MCU
Parts:
- removed D81, D82, D83, D84, D85, D86, D87, D90, D95, D96: ~, Diode_THT:D_DO-35_SOD27_P7.62mm_Horizontal
- added D10: ~, Diode_THT:D_DO-35_SOD27_P7.62mm_Horizontal, F.Cu at (377.7, 133.2)
- added D14: ~, Diode_THT:D_DO-35_SOD27_P7.62mm_Horizontal, F.Cu at (403.9, 101.3)
- added D16: ~, Diode_THT:D_DO-35_SOD27_P7.62mm_Horizontal, F.Cu at (399.1, 108.4)
- added D21: ~, Diode_THT:D_DO-35_SOD27_P7.62mm_Horizontal, F.Cu at (392.0, 126.2)
- added D36: ~, Diode_THT:D_DO-35_SOD27_P7.62mm_Horizontal, F.Cu at (413.4, 129.8)
- added D37: ~, Diode_THT:D_DO-35_SOD27_P7.62mm_Horizontal, F.Cu at (415.8, 133.3)
- added D48: ~, Diode_THT:D_DO-35_SOD27_P7.62mm_Horizontal, F.Cu at (427.7, 122.7)
- added D60: ~, Diode_THT:D_DO-35_SOD27_P7.62mm_Horizontal, F.Cu at (384.8, 165.1)
- added D77: ~, Diode_THT:D_DO-35_SOD27_P7.62mm_Horizontal, F.Cu at (434.8, 158.1)
- added D78: ~, Diode_THT:D_DO-35_SOD27_P7.62mm_Horizontal, F.Cu at (437.2, 161.7)
- C1: renamed from C7; moved to B.Cu
- C2: renamed from C8; moved to B.Cu
- C3: renamed from C9; moved to B.Cu
- C4: renamed from C1; moved to B.Cu
- C5: renamed from C2; moved to B.Cu
- C6: renamed from C3; moved to B.Cu
- C7: renamed from C4; moved to B.Cu
- C8: renamed from C5; moved to B.Cu
- C9: renamed from C6; moved to B.Cu
- ESDProtection1, F1, J2, ResetSW1, VoltStepDown1: moved to B.Cu
- R1: renamed from R3; moved to B.Cu
- R2: renamed from R1; moved to B.Cu
- R3: renamed from R2; moved to B.Cu
- U1: renamed from U2; footprint Package_QFP:LQFP-48_7x7mm_P0.5mm -> Keebio-Parts.pretty-master:LQFP-48_7x7mm_Pitch0.5mm; moved to B.Cu
- moved C1 504.8 mm to (98.1, 101.9), turned to 90 degrees
- moved C9 503.4 mm to (94.0, 101.9), turned to -90 degrees
- moved C8 501.9 mm to (96.0, 101.9), turned to -90 degrees
- moved R2 501.4 mm to (96.4, 77.7), turned to 180 degrees
- moved C4 499.7 mm to (92.1, 88.7), turned to 180 degrees
- moved C7 495.9 mm to (102.2, 99.4), turned to -90 degrees
- moved C2 495.4 mm to (104.2, 84.0), turned to -90 degrees
- moved R3 493.9 mm to (103.7, 77.7)
- moved F1 490.5 mm to (103.8, 80.3), turned to 180 degrees
- moved R1 490.2 mm to (109.4, 98.4), turned to 180 degrees
- moved ESDProtection1 489.8 mm to (100.0, 83.8), turned to 90 degrees
- moved C5 488.6 mm to (102.9, 88.4)
- moved C3 488.2 mm to (112.2, 91.8)
- moved C6 487.4 mm to (105.0, 97.5)
- moved U1 485.0 mm to (98.0, 93.4), turned to 90 degrees
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- renumbered SW11 to SW1, SW9 to SW10, SW10 to SW11, SW1 to SW2, SW2 to SW3, SW3 to SW4, SW4 to SW5, SW5 to SW6, SW6 to SW7, SW7 to SW8, SW8 to SW9
Connections:
- D11 pad 1: Row 2 -> Row 0
- D12 pad 1: Row 2 -> Row 0
- D13 pad 1: Row 3 -> Row 0
- D15 pad 1: Row 5 -> Row 1
- D17 pad 1: Row 4 -> Row 1
- D18 pad 1: Row 5 -> Row 1
- D19 pad 1: Row 3 -> Row 1
- D2 pad 1: Row 5 -> Row 0
- D20 pad 1: Row 4 -> Row 1
- D22 pad 1: Row 3 -> Row 1
- D23 pad 1: Row 4 -> Row 1
- D24 pad 1: Row 5 -> Row 1
- D25 pad 1: Row 0 -> Row 1
- D27 pad 1: Row 2 -> Row 1
- D28 pad 1: Row 3 -> Row 2
- D29 pad 1: Row 4 -> Row 2
- D30 pad 1: Row 5 -> Row 2
- D31 pad 1: Row 0 -> Row 2
- D32 pad 1: Row 1 -> Row 2
- D34 pad 1: Row 3 -> Row 2
- D35 pad 1: Row 4 -> Row 2
- D38 pad 1: Row 1 -> Row 2
- D40 pad 1: Row 3 -> Row 2
- D41 pad 1: Row 4 -> Row 2
- D42 pad 1: Row 5 -> Row 3
- D43 pad 1: Row 0 -> Row 3
- D44 pad 1: Row 1 -> Row 3
- D45 pad 1: Row 2 -> Row 3
- D47 pad 1: Row 4 -> Row 3
- D49 pad 1: Row 0 -> Row 3
- D5 pad 1: Row 1 -> Row 0
- D50 pad 1: Row 1 -> Row 3
- D51 pad 1: Row 2 -> Row 3
- D53 pad 1: Row 4 -> Row 3
- D54 pad 1: Row 5 -> Row 3
- D55 pad 1: Row 0 -> Row 4
- D56 pad 1: Row 1 -> Row 4
- D57 pad 1: Row 2 -> Row 4
- D58 pad 1: Row 3 -> Row 4
- D6 pad 1: Row 1 -> Row 0
- D61 pad 1: Row 0 -> Row 4
- D62 pad 1: Row 1 -> Row 4
- D63 pad 1: Row 2 -> Row 4
- D64 pad 1: Row 3 -> Row 4
- D66 pad 1: Row 5 -> Row 4
- D67 pad 1: Row 0 -> Row 4
- D68 pad 1: Row 1 -> Row 5
- D69 pad 1: Row 2 -> Row 5
- D7 pad 1: Row 1 -> Row 0
- D70 pad 1: Row 3 -> Row 5
- D71 pad 1: Row 4 -> Row 5
- D73 pad 1: Row 0 -> Row 5
- D74 pad 1: Row 1 -> Row 5
- D75 pad 1: Row 2 -> Row 5
- D76 pad 1: Row 3 -> Row 5
- D79 pad 1: Row 0 -> Row 5
- D8 pad 1: Row 1 -> Row 0
- D9 pad 1: Row 2 -> Row 0
- ESDProtection1 pad 4: Net-(ESDProtection1-I/O2-Pad4) -> D-
- ESDProtection1 pad 6: Net-(ESDProtection1-I/O1-Pad6) -> D+
- J2 pad A6: Net-(ESDProtection1-I/O1-Pad6) -> D+
- J2 pad A7: Net-(ESDProtection1-I/O2-Pad4) -> D-
- J2 pad B6: Net-(ESDProtection1-I/O1-Pad6) -> D+
- J2 pad B7: Net-(ESDProtection1-I/O2-Pad4) -> D-
- SW+1 pad 2: Net-(D74-A) -> Net-(D26-A)
- SW-1 pad 2: Net-(D68-A) -> Net-(D25-A)
- SW10 pad 2: Net-(D56-A) -> Net-(D23-A)
- SW11 pad 2: Net-(D62-A) -> Net-(D24-A)
- SW2 pad 2: Net-(D6-A) -> Net-(D15-A)
- SW3 pad 2: Net-(D7-A) -> Net-(D16-A)
- SW4 pad 2: Net-(D8-A) -> Net-(D17-A)
- SW5 pad 2: Net-(D26-A) -> Net-(D18-A)
- SW6 pad 2: Net-(D32-A) -> Net-(D19-A)
- SW7 pad 2: Net-(D38-A) -> Net-(D20-A)
- SW8 pad 2: Net-(D44-A) -> Net-(D21-A)
- SW9 pad 2: Net-(D50-A) -> Net-(D22-A)
- SWBckspc2u1 pad 2: Net-(D86-A) -> Net-(D27-A)
- SWCaplck1.75u1 pad 2: Net-(D13-A) -> Net-(D42-A)
- SWDel1 pad 2: Net-(D84-A) -> Net-(D76-A)
- SWEnter2.25u1 pad 2: Net-(D82-A) -> Net-(D54-A)
- SWF1 pad 2: Net-(D3-A) -> Net-(D2-A)
- SWF10 pad 2: Net-(D73-A) -> Net-(D11-A)
- SWF11 pad 2: Net-(D79-A) -> Net-(D12-A)
- SWF12 pad 2: Net-(D85-A) -> Net-(D13-A)
- SWF2 pad 2: Net-(D4-A) -> Net-(D3-A)
- SWF3 pad 2: Net-(D25-A) -> Net-(D4-A)
- SWF4 pad 2: Net-(D31-A) -> Net-(D5-A)
- SWF5 pad 2: Net-(D43-A) -> Net-(D6-A)
- SWF6 pad 2: Net-(D49-A) -> Net-(D7-A)
- SWF7 pad 2: Net-(D55-A) -> Net-(D8-A)
- SWF8 pad 2: Net-(D61-A) -> Net-(D9-A)
- SWF9 pad 2: Net-(D67-A) -> Net-(D10-A)
- SWLCtrl1.25u1 pad 2: Net-(D15-A) -> Net-(D68-A)
- SWLalt1.25u1 pad 2: Net-(D24-A) -> Net-(D70-A)
- SWLshift2.25u1 pad 2: Net-(D17-A) -> Net-(D55-A)
- SWLwin1.25u1 pad 2: Net-(D18-A) -> Net-(D69-A)
- SWRalt1.25u1 pad 2: Net-(D66-A) -> Net-(D74-A)
- SWRight1 pad 2: Net-(D2-A) -> Net-(D79-A)
- SWRshift2.25u1 pad 2: Net-(D83-A) -> Net-(D66-A)
- SWRwin1.25u1 pad 2: Net-(D72-A) -> Net-(D75-A)
- SWSpc1.25u1 pad 2: Net-(D42-A) -> Net-(D72-A)
- SWSpc2.25u1 pad 2: Net-(D30-A) -> Net-(D71-A)
- SWSpc2.75u1 pad 2: Net-(D54-A) -> Net-(D73-A)
- SWTab1.5u1 pad 2: Net-(D9-A) -> Net-(D28-A)
- SWUp1 pad 2: Net-(D95-A) -> Net-(D67-A)
- SW_'1 pad 2: Net-(D76-A) -> Net-(D53-A)
- SW_,1 pad 2: Net-(D59-A) -> Net-(D63-A)
- SW_.1 pad 2: Net-(D65-A) -> Net-(D64-A)
- SW_/1 pad 2: Net-(D71-A) -> Net-(D65-A)
- SW_;1 pad 2: Net-(D70-A) -> Net-(D52-A)
- SW_A1 pad 2: Net-(D19-A) -> Net-(D43-A)
- SW_B1 pad 2: Net-(D41-A) -> Net-(D60-A)
- SW_C1 pad 2: Net-(D29-A) -> Net-(D58-A)
- SW_D1 pad 2: Net-(D28-A) -> Net-(D45-A)
- SW_E1 pad 2: Net-(D27-A) -> Net-(D31-A)
- SW_F1 pad 2: Net-(D34-A) -> Net-(D46-A)
- SW_G1 pad 2: Net-(D40-A) -> Net-(D47-A)
- SW_H1 pad 2: Net-(D46-A) -> Net-(D48-A)
- SW_I1 pad 2: Net-(D57-A) -> Net-(D36-A)
- SW_J1 pad 2: Net-(D52-A) -> Net-(D49-A)
- SW_K1 pad 2: Net-(D58-A) -> Net-(D50-A)
- SW_L1 pad 2: Net-(D64-A) -> Net-(D51-A)
- SW_M1 pad 2: Net-(D53-A) -> Net-(D62-A)
- SW_N1 pad 2: Net-(D47-A) -> Net-(D61-A)
- SW_O1 pad 2: Net-(D63-A) -> Net-(D37-A)
- SW_P1 pad 2: Net-(D69-A) -> Net-(D38-A)
- SW_Q1 pad 2: Net-(D11-A) -> Net-(D29-A)
- SW_R1 pad 2: Net-(D33-A) -> Net-(D32-A)
- SW_S1 pad 2: Net-(D22-A) -> Net-(D44-A)
- SW_T1 pad 2: Net-(D39-A) -> Net-(D33-A)
- SW_U1 pad 2: Net-(D51-A) -> Net-(D35-A)
- SW_V1 pad 2: Net-(D35-A) -> Net-(D59-A)
- SW_W1 pad 2: Net-(D12-A) -> Net-(D30-A)
- SW_X1 pad 2: Net-(D23-A) -> Net-(D57-A)
- SW_Y1 pad 2: Net-(D45-A) -> Net-(D34-A)
- SW_Z1 pad 2: Net-(D20-A) -> Net-(D56-A)
- SW_[1 pad 2: Net-(D75-A) -> Net-(D39-A)
- SW_\1.5u1 pad 2: Net-(D87-A) -> Net-(D41-A)
- SW_]1 pad 2: Net-(D81-A) -> Net-(D40-A)
- SW`1 pad 2: Net-(D5-A) -> Net-(D14-A)
- U1 pad 10: Row 0 -> Col 9
- U1 pad 11: Row 1 -> Col 8
- U1 pad 12: Row 2 -> Col 7
- U1 pad 16: unconnected-(U2-PA6-Pad16) -> Col 6
- U1 pad 17: unconnected-(U2-PA7-Pad17) -> Col 5
- U1 pad 18: Col 3 -> Col 4
- U1 pad 19: Col 4 -> Col 3
- U1 pad 2: Col 0 -> Row 0
- U1 pad 20: Col 5 -> Col 2
- U1 pad 21: Col 13 -> Col 1
- U1 pad 22: Col 14 -> Col 0
- U1 pad 29: RotaryA -> unconnected-(U1-PA8-Pad29)
- U1 pad 3: Col 1 -> Row 1
- U1 pad 30: RotaryB -> unconnected-(U1-PA9-Pad30)
- U1 pad 39: Col 6 -> RotaryA
- U1 pad 4: Col 2 -> Row 2
- U1 pad 40: Col 7 -> RotaryB
- U1 pad 41: Col 8 -> Col 14
- U1 pad 42: Col 9 -> Col 13
- U1 pad 43: Col 10 -> Col 12
- U1 pad 46: Col 12 -> Col 10
Routing:
- net Col 16: track 0.00 -> 443.6 mm
- net Col 15: track 0.00 -> 442.6 mm
- net Net-(D68-A): track 0.00 -> 383.0 mm
- net Col 13: track 0.00 -> 358.2 mm
- net Net-(D69-A): track 0.00 -> 354.1 mm
- net Col 14: track 0.00 -> 352.6 mm
- net Net-(D70-A): track 0.00 -> 322.8 mm
- net Net-(D1-A): track 0.00 -> 317.7 mm
- net Col 11: track 0.00 -> 305.1 mm
- net Col 10: track 0.00 -> 289.8 mm
- net Net-(D71-A): track 0.00 -> 288.6 mm
- net Col 8: track 0.00 -> 282.5 mm
- net Net-(D2-A): track 0.00 -> 281.5 mm
- net Col 9: track 0.00 -> 281.4 mm
- net Col 12: track 0.00 -> 280.4 mm
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Other:
- board outline added: 376.2 x 128.6 mm

Commit message: Added more traces
Routing:
- net Row 3: track 54.4 -> 536.2 mm, vias 0 -> 4
- net Row 5: track 65.6 -> 450.7 mm, vias 0 -> 2
- net Row 2: track 58.9 -> 422.4 mm, vias 0 -> 2
- net Net-(D14-A): track 0.00 -> 353.5 mm
- net Net-(D15-A): track 0.00 -> 346.0 mm
- net Row 4: track 67.9 -> 412.0 mm, vias 0 -> 2
- net Row 1: track 59.2 -> 399.1 mm, vias 0 -> 2
- net Net-(D16-A): track 0.00 -> 320.2 mm
- net Row 0: track 54.4 -> 374.4 mm, vias 0 -> 2
- net Net-(D17-A): track 0.00 -> 299.7 mm
- net Net-(D55-A): track 0.00 -> 291.6 mm, vias 0 -> 1
- net Net-(D18-A): track 0.00 -> 283.8 mm
- net Net-(D19-A): track 0.00 -> 267.5 mm
- net Net-(D20-A): track 0.00 -> 261.1 mm
- net Net-(D56-A): track 0.00 -> 255.3 mm
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
Commit message: Changed diodes and redoing matrix
Parts:
- moved D1 301.0 mm to (83.8, 99.0), turned to 90 degrees
- moved D2 260.8 mm to (121.7, 99.0), turned to 90 degrees
- moved D3 239.5 mm to (140.7, 99.0), turned to 90 degrees
- moved D4 218.5 mm to (159.6, 99.0), turned to 90 degrees
- moved D5 197.0 mm to (179.0, 99.0), turned to 90 degrees
- moved D6 166.8 mm to (207.3, 99.0), turned to 90 degrees
- moved D7 145.9 mm to (226.6, 99.0), turned to 90 degrees
- moved D8 130.3 mm to (245.5, 99.0), turned to 90 degrees
- moved D9 114.9 mm to (264.6, 99.0), turned to 90 degrees
- moved D10 91.5 mm to (292.9, 99.0), turned to 90 degrees
- moved D11 77.6 mm to (312.3, 99.0), turned to 90 degrees
- moved D12 65.7 mm to (331.5, 99.0), turned to 90 degrees
- moved D54 61.0 mm to (381.0, 147.2), turned to -90 degrees
- moved D13 56.7 mm to (350.2, 99.0), turned to 90 degrees
- moved D53 54.1 mm to (385.8, 146.0), turned to -90 degrees
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Routing:
- net Row 3: track 536.2 -> 62.9 mm, vias 4 -> 0
- net Col 16: track 443.6 -> 0.00 mm
- net Col 15: track 442.6 -> 19.0 mm
- net Row 5: track 450.7 -> 52.4 mm, vias 2 -> 0
- net Net-(D28-A): track 0.00 -> 363.6 mm
- net Net-(D42-A): track 0.00 -> 356.4 mm
- net Row 2: track 422.4 -> 68.2 mm, vias 2 -> 0
- net Net-(D14-A): track 353.5 -> 0.00 mm
- net Row 4: track 412.0 -> 63.5 mm, vias 2 -> 0
- net Net-(D15-A): track 346.0 -> 0.00 mm
- net Net-(D29-A): track 0.00 -> 335.1 mm
- net Row 1: track 399.1 -> 68.4 mm, vias 2 -> 0
- net Net-(D43-A): track 0.00 -> 325.6 mm
- net Net-(D16-A): track 320.2 -> 0.00 mm
- net Net-(D30-A): track 0.00 -> 311.5 mm
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Other:
- board text added: "D10"

Commit message: Finished traces
Connections:
- U1 pad 10: Col 9 -> unconnected-(U1-PA0-Pad10)
- U1 pad 11: Col 8 -> unconnected-(U1-PA1-Pad11)
- U1 pad 12: Col 7 -> unconnected-(U1-PA2-Pad12)
- U1 pad 13: Row 3 -> Row 5
- U1 pad 15: Row 5 -> Row 3
- U1 pad 16: Col 6 -> Col 1
- U1 pad 17: Col 5 -> Col 2
- U1 pad 19: Col 3 -> Col 5
- U1 pad 20: Col 2 -> Col 6
- U1 pad 21: Col 1 -> Col 3
- U1 pad 25: Col 15 -> Col 16
- U1 pad 26: Col 16 -> Col 15
- U1 pad 27: unconnected-(U1-PB14-Pad27) -> RotaryA
- U1 pad 28: unconnected-(U1-PB15-Pad28) -> RotaryB
- U1 pad 29: unconnected-(U1-PA8-Pad29) -> Oled2
- U1 pad 30: unconnected-(U1-PA9-Pad30) -> Oled1
- U1 pad 37: Oled1 -> unconnected-(U1-PA14-Pad37)
- U1 pad 38: Oled2 -> Col 7
- U1 pad 39: RotaryA -> Col 8
- U1 pad 40: RotaryB -> Col 9
- U1 pad 41: Col 14 -> Col 10
- U1 pad 42: Col 13 -> Col 11
- U1 pad 45: Col 11 -> Col 13
- U1 pad 46: Col 10 -> Col 14
Routing:
- net Row 3: track 62.9 -> 520.8 mm, vias 0 -> 3
- net Row 4: track 63.5 -> 504.7 mm, vias 0 -> 3
- net Row 5: track 52.4 -> 493.4 mm, vias 0 -> 3
- net Col 16: track 0.00 -> 434.3 mm, vias 0 -> 1
- net Col 15: track 19.0 -> 436.1 mm
- net RotaryA: track 0.00 -> 379.9 mm
- net Net-(D14-A): track 0.00 -> 378.9 mm
- net RotaryB: track 0.00 -> 369.8 mm
- net GND: track 0.00 -> 358.6 mm, vias 0 -> 12
- net Net-(D15-A): track 0.00 -> 356.5 mm, vias 0 -> 2
- net RotarySW: track 0.00 -> 351.7 mm
- net Net-(D16-A): track 0.00 -> 333.2 mm
- net +3.3V: track 32.9 -> 353.9 mm, vias 0 -> 4
- net Oled2: track 0.00 -> 317.1 mm, vias 0 -> 1
- net Oled1: track 0.00 -> 314.2 mm, vias 0 -> 1
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- added copper zone on B.Cu, net GND
- added copper zone on F.Cu, net GND
