File: Keyboard Designs/Schematics/75TH/75TH/75TH.kicad_sch (KiCad schematic)
At the start: 14 parts, among them J1 OLED_128x64, J2 USB_C_Receptacle_USB2.0_14P, SW11 RotaryEncoder_Switch, U2 STM32F072CBTx

Commit message: Started pcb layout
Parts:
- added C8, C9: 10uF, Capacitor_SMD:C_0805_2012Metric, symbol Device:C
- added ESDProtection1: USBLC6-2SC6, Package_TO_SOT_SMD:SOT-23-6, symbol Power_Protection:USBLC6-2SC6
- added R3: 10k, ScottoKeebs_Components:Resistor_0805, symbol ScottoKeebs:Placeholder_Resistor
- added ResetSW1: Switch, Button_Switch_SMD:SW_SPST_SKQG_WithStem, symbol ScottoKeebs:Placeholder_Switch
- added VoltStepDown1: AMS1117-3.3, Package_TO_SOT_SMD:SOT-223-3_TabPin2, symbol Regulator_Linear:AMS1117-3.3
- C1, C2, C3, C4, C5, C6, C7: footprint (none) -> Capacitor_SMD:C_0805_2012Metric
- F1: footprint (none) -> ScottoKeebs_Components:Fuse_0603
- J2: footprint (none) -> Connector_USB:USB_C_Receptacle_HRO_TYPE-C-31-M-12
- R1, R2: footprint (none) -> ScottoKeebs_Components:Resistor_0805
- SW11: value RotaryEncoder_Switch -> RotaryEncoder_Switch_EC11E09244AQ
Connections:
- net +3.3V: now also J1.2 (VCC), C9.1, ResetSW1.1, VoltStepDown1.2 (VO)
- net +5V: now also C8.1, ESDProtection1.5 (VBUS), VoltStepDown1.3 (VI)
- net D+: now also ESDProtection1.1 (I/O1); no longer J2.A6 (D+), J2.B6 (D+)
- net D-: now also ESDProtection1.3 (I/O2); no longer J2.A7 (D-), J2.B7 (D-)
- net GND: now also J1.1 (GND), SW11.C, SW11.S2, C8.2, C9.2, ESDProtection1.2 (GND), R3.2, VoltStepDown1.1 (GND)
- net VBUS: now reaches F1.1, J2.A4 (VBUS), J2.A9 (VBUS), J2.B4 (VBUS), J2.B9 (VBUS)
- net Oled1: now reaches J1.3 (SCL)
- net Oled1: now also U2.37 (PA14)
- net Oled2: now reaches J1.4 (SDA)
- net Oled2: now also U2.38 (PA15)
- net RotaryA: now reaches U2.29 (PA8)
- net RotaryA: now also SW11.A
- net RotaryB: now reaches U2.30 (PA9)
- net RotaryB: now also SW11.B
- net RotarySW: now reaches U2.31 (PA10)
- net RotarySW: now also SW11.S1
- net BOOT0: now reaches U2.44 (BOOT0)
- net BOOT0: now also R3.1, ResetSW1.2
- net Col 17: no longer names the net of U2.27 (PB14)
- new net: ESDProtection1.4 (I/O2), J2.A7 (D-), J2.B7 (D-)
- new net: ESDProtection1.6 (I/O1), J2.A6 (D+), J2.B6 (D+)
- no-connect marks 0 -> 7
Other:
- moved on the sheet: J1, SW11

Commit message: wired usbc and partial MCU
Parts:
- U1: renamed from U2; footprint Package_QFP:LQFP-48_7x7mm_P0.5mm -> Keebio-Parts.pretty-master:LQFP-48_7x7mm_Pitch0.5mm
- renumbered C7 to C1, C8 to C2, C9 to C3, C1 to C4, C2 to C5, C3 to C6, C4 to C7, C5 to C8, C6 to C9, R3 to R1, R1 to R2, R2 to R3, SW11 to SW1
Connections:
- net Col 0: now also U1.22 (PB11); no longer U1.2 (PC13)
- net Col 1: now also U1.21 (PB10); no longer U1.3 (PC14)
- net Col 10: now also U1.46 (PB9); no longer U1.43 (PB7)
- net Col 12: now also U1.43 (PB7); no longer U1.46 (PB9)
- net Col 13: now also U1.42 (PB6); no longer U1.21 (PB10)
- net Col 14: now also U1.41 (PB5); no longer U1.22 (PB11)
- net Col 2: now also U1.20 (PB2); no longer U1.4 (PC15)
- net Col 3: now also U1.19 (PB1); no longer U1.18 (PB0)
- net Col 4: now also U1.18 (PB0); no longer U1.19 (PB1)
- net Col 5: now also U1.17 (PA7); no longer U1.20 (PB2)
- net Col 6: now also U1.16 (PA6); no longer U1.39 (PB3)
- net Col 7: now also U1.12 (PA2); no longer U1.40 (PB4)
- net Col 8: now also U1.11 (PA1); no longer U1.41 (PB5)
- net Col 9: now also U1.10 (PA0); no longer U1.42 (PB6)
- net D+: now also ESDProtection1.6 (I/O1), J2.A6 (D+), J2.B6 (D+)
- net D-: now also ESDProtection1.4 (I/O2), J2.A7 (D-), J2.B7 (D-)
- net RotaryA: now also U1.39 (PB3); no longer U1.29 (PA8)
- net RotaryB: now also U1.40 (PB4); no longer U1.30 (PA9)
- net Row 0: now also U1.2 (PC13); no longer U1.10 (PA0)
- net Row 1: now also U1.3 (PC14); no longer U1.11 (PA1)
- net Row 2: now also U1.4 (PC15); no longer U1.12 (PA2)
Other:
- moved on the sheet: ESDProtection1

Commit message: Finished traces
Connections:
- net Col 1: now also U1.16 (PA6); no longer U1.21 (PB10)
- net Col 10: now also U1.41 (PB5); no longer U1.46 (PB9)
- net Col 11: now also U1.42 (PB6); no longer U1.45 (PB8)
- net Col 13: now also U1.45 (PB8); no longer U1.42 (PB6)
- net Col 14: now also U1.46 (PB9); no longer U1.41 (PB5)
- net Col 15: now also U1.26 (PB13); no longer U1.25 (PB12)
- net Col 16: now also U1.25 (PB12); no longer U1.26 (PB13)
- net Col 2: now also U1.17 (PA7); no longer U1.20 (PB2)
- net Col 3: now also U1.21 (PB10); no longer U1.19 (PB1)
- net Col 5: now also U1.19 (PB1); no longer U1.17 (PA7)
- net Col 6: now also U1.20 (PB2); no longer U1.16 (PA6)
- net Col 7: now also U1.38 (PA15); no longer U1.12 (PA2)
- net Col 8: now also U1.39 (PB3); no longer U1.11 (PA1)
- net Col 9: now also U1.40 (PB4); no longer U1.10 (PA0)
- net Oled1: now also U1.30 (PA9); no longer U1.37 (PA14)
- net Oled2: now also U1.29 (PA8); no longer U1.38 (PA15)
- net RotaryA: now also U1.27 (PB14); no longer U1.39 (PB3)
- net RotaryB: now also U1.28 (PB15); no longer U1.40 (PB4)
- net Row 3: now also U1.15 (PA5); no longer U1.13 (PA3)
- net Row 5: now also U1.13 (PA3); no longer U1.15 (PA5)
